Commit message: feat: real-robot navigation bring-up, firmware false-positive fixes, calibration tools
Firmware (ESP32-S3 base control)
- relax stall detection: STALL_SPEED 4 mm/s, floor 12% of demand, 2.0 s window
  (previously 8 mm/s / 25% / 0.8 s made any command >80 mm/s trip BASE_STALL)
- relax overspeed: 700 mm/s over 0.4 s (wheel slip on tile exceeded 420 mm/s)
- keep MAX_DUTY .90 / BASE_DUTY .60 / ramp .5
- update host tests for the new thresholds

base_bridge
- heading hold on the manual path (IMU yaw, gain 1.5, clamp 0.12 rad/s)
- sensor_timeout_s 0.5 wired into scan/IMU watchdogs
- ignore explore "stopped" while a nav goal is active (two-point handover)
- 3 s debounce before disarming on explore-stopped
- clearer clear-fault messages (no fault vs stale serial state)

Nav2 / costs
- global inflation 0.30 -> 0.20 to fit the 0.86 m doorway (0.86 - 2R > 0.43 m)
- local inflation 0.20 with footprint clearing
- front_stop half width 0.24 m, 3 points required (single noisy point froze the robot)
- behavior_server simulate_ahead_time 0.5 s (2.0 s aborted spins near walls)
- rotation shim angular_dist_threshold 0.6 rad (turn first in tight spots)

Odometry / SLAM
- wheel track 0.268 m, circumference 0.2012 m (hand push 1.000 m -> 0.993 m)
- EKF fuses wheel vx only, IMU absolute yaw + gyro rate
- slam_toolbox crash-safe mapping params (minimum_travel_* 0.5)
- Cartographer and RTAB-Map launch/config alternatives

Tools and docs
- odom/track calibration, AMCL seeding, map save/pause/rollback/health,
  fault reset, keyboard helper
- docs/AGENT_LOG.md session log, mapping workflow + step-by-step runbook,
  hardware notes, RViz panel sources
- maps: 2026-10-28/29 scans including the edited navigation map

Repo hygiene
- ignore *.bak, slam_toolbox serialization, third-party checkouts
  (their local patches are kept under patches/)

File: ros2_ws/src/fwr_bringup/description/fwr_chassis_demo.urdf (robot description, URDF)
Before this commit: robot fwr_chassis_preview, 8 links, 7 joints
Links:
- added link base_footprint
- added link imu_link
- added link left_motor_bracket, mass 0.4; visual mesh filename=package://fwr_bringup/description/mg513x_motor_bracket.stl
- added link motor_driver_body, mass 0.08; collision box size=0.050 0.055 0.014; visual mesh filename=package://fwr_bringup/description/at8236_d157b.stl
- added link right_motor_bracket, mass 0.4; visual mesh filename=package://fwr_bringup/description/mg513x_motor_bracket.stl
- link base_link: mass None -> 5; geometry collision box size=0.52 0.35 0.16; visual mesh filename=package://fwr_bringup/description/fwr_chassis_wheel_recesse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
- link front_left_caster_swivel: mass None -> 0.05
- link front_left_caster_wheel: mass None -> 0.08
- link front_right_caster_swivel: mass None -> 0.05
- link front_right_caster_wheel: mass None -> 0.08
- link laser_front: geometry collision box size=0.0556 0.0556 0.0413; visual mesh filename=package://fwr_bringup/description/rplidar_c1_cad.stl
- link left_drive_wheel: mass None -> 0.25; geometry collision cylinder length=0.035 radius=0.0325; visual cylinder length=0.035 radius=0.0325
- link right_drive_wheel: mass None -> 0.25; geometry collision cylinder length=0.035 radius=0.0325; visual cylinder length=0.035 radius=0.0325
Joints:
- added joint base_footprint_joint: type fixed, parent base_footprint, child base_link, origin xyz=0 0 0.0325
- added joint imu_frame_joint: type fixed, parent base_link, child imu_link, origin xyz=0 0 0
- added joint left_motor_mount_joint: type fixed, parent base_link, child left_motor_bracket, origin xyz=-0.13 0.08 0.0175
- added joint motor_driver_mount_joint: type fixed, parent base_link, child motor_driver_body, origin xyz=-0.07 0 0.1745
- added joint right_motor_mount_joint: type fixed, parent base_link, child right_motor_bracket, origin xyz=-0.13 -0.08 0.0175 rpy=0 0 3.14159265359
- joint front_left_caster_steer_joint: origin xyz=0.19 0.115 0.09 -> xyz=0.19 0.115 0.0575
- joint front_right_caster_steer_joint: origin xyz=0.19 -0.115 0.09 -> xyz=0.19 -0.115 0.0575
- joint laser_front_joint: origin xyz=0.19 0 0.2298 rpy=0 0 0 -> xyz=0.21 0 0.0425 rpy=0 0 3.14159265359
- joint left_drive_wheel_preview_joint: origin xyz=-0.13 0.145 0.05 -> xyz=-0.13 0.1575 0
- joint right_drive_wheel_preview_joint: origin xyz=-0.13 -0.145 0.05 -> xyz=-0.13 -0.1575 0
